File: carte/duobot/duobot.kicad_pcb (KiCad board)
At the start: 2 copper layers, 100 x 70 mm, 28 parts, among them J1 Moteur Gauche, J2 Moteur Droite, J3 MPU6050, J4 HC-05 BT, J5 Batterie, J6 Extension, X1 Trou, X2 Trou, X3 Trou, X4 Trou

Commit message: Finalisation routage et schéma
Parts:
- removed J3: MPU6050, Connector_PinHeader_1.00mm:PinHeader_1x08_P1.00mm_Vertical
- removed J6: Extension, Connector_PinHeader_1.00mm:PinHeader_1x10_P1.00mm_Vertical
- added J2: Extension, Connector_PinHeader_2.54mm:PinHeader_2x05_P2.54mm_Vertical, F.Cu at (117.0, 68.5)
- added U1: ~, bpc:BPC_MPU6050, F.Cu at (113.2, 107.0)
- J4: value HC-05 BT -> HC05 - BT; footprint Connector_PinHeader_1.00mm:PinHeader_1x06_P1.00mm_Vertical -> Connector_PinHeader_2.54mm:PinHeader_1x06_P2.54mm_Vertical
- moved J4 3.64 mm to (155.0, 115.0)
- moved R1 3.61 mm to (99.4, 85.0)
- moved R2 2.50 mm to (114.6, 110.5)
Routing:
- net +5V: track 157.6 -> 169.5 mm
- net A7: track 24.5 -> 34.7 mm, vias 0 -> 2
- net A6: track 23.0 -> 29.0 mm, vias 0 -> 2
- net SDA: track 22.1 -> 27.5 mm, vias 0 -> 1
- net SCL: track 25.6 -> 29.0 mm, vias 0 -> 1
- net Net-(A3-VDD): track 58.7 -> 61.6 mm
- net A2: track 15.0 -> 12.1 mm
- net A3: track 16.1 -> 18.8 mm, vias 0 -> 2
- net D12: track 49.6 -> 47.5 mm
- net D2: track 78.7 -> 80.1 mm
- net A1: track 13.7 -> 12.4 mm
- net Net-(A1-D0/RX): track 12.9 -> 14.2 mm
Other:
- board text added: "Carte de pilotage pour 2 moteurs"
- board text added: "Extension"
- board text added: "HC05 BT - Télécommande"
- board text removed: "Carte de pilotage 2 moteurs"
- board text removed: "EXTENSION"
- board text removed: "MPU 6050"

Commit message: Correction suite analyse des règles PCB
Routing:
- net M2: track 66.8 -> 65.7 mm
- net +5V: track 169.5 -> 168.5 mm
- net Net-(A3-VDD): vias 1 -> 0
Other:
- board text added: "Télécommande"
- board text removed: "HC05 BT - Télécommande"
Changed lines of the file:
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@@
     (property "ki_keywords" "connector")
     (attr through_hole)
-    (fp_text reference "J4" (at 3 0.04) (layer "F.SilkS")
+    (fp_text reference "J4" (at 0 15.54) (layer "F.SilkS")
         (effects (font (size 1 1) (thickness 0.15)))
     )
@@
     (effects (font (size 1 1) (thickness 0.15)) (justify left bottom))
   )
-  (gr_text "HC05 BT - Télécommande" (at 141.75 113) (layer "F.SilkS")
+  (gr_text "Télécommande" (at 144 113) (layer "F.SilkS")
     (effects (font (size 0.9 0.9) (thickness 0.15)) (justify left bottom))
   )
@@
     (effects (font (size 1 1) (thickness 0.15)) (justify left bottom))
   )
-  (gr_text "HC-05 BT" (at 146 116) (layer "F.SilkS")
+  (gr_text "HC-05 BT" (at 143.5 117.75) (layer "F.SilkS")
     (effects (font (size 1 1) (thickness 0.125) bold) (justify left bottom))
   )
@@
   (segment (start 152 79) (end 143.06 79) (width 0.25) (layer "F.Cu") (net 9))
   (via (at 166.5 103) (size 0.8) (drill 0.4) (layers "F.Cu" "B.Cu") (net 9))
-  (segment (start 163 115.84) (end 166.66 115.84) (width 0.25) (layer "B.Cu") (net 9))
-  (segment (start 168 114.5) (end 168 104.5) (width 0.25) (layer "B.Cu") (net 9))
-  (segment (start 168 104.5) (end 166.5 103) (width 0.25) (layer "B.Cu") (net 9))
-  (segment (start 166.66 115.84) (end 168 114.5) (width 0.25) (layer "B.Cu") (net 9))
+  (segment (start 164.75 115.25) (end 164.16 115.84) (width 0.25) (layer "B.Cu") (net 9))
+  (segment (start 165.25 114) (end 164.75 114.5) (width 0.25) (layer "B.Cu") (net 9))
+  (segment (start 167.25 108.75) (end 167.25 112.5) (width 0.25) (layer "B.Cu") (net 9))
+  (segment (start 168 104.5) (end 168 108) (width 0.25) (layer "B.Cu") (net 9))
+  (segment (start 168 108) (end 167.25 108.75) (width 0.25) (layer "B.Cu") (net 9))
+  (segment (start 165.75 114) (end 165.25 114) (width 0.25) (layer "B.Cu") (net 9))
+  (segment (start 164.75 114.5) (end 164.75 115.25) (width 0.25) (layer "B.Cu") (net 9))
+  (segment (start 166.5 103) (end 168 104.5) (width 0.25) (layer "B.Cu") (net 9))
+  (segment (start 167.25 112.5) (end 165.75 114) (width 0.25) (layer "B.Cu") (net 9))
+  (segment (start 164.16 115.84) (end 163 115.84) (width 0.25) (layer "B.Cu") (net 9))
   (segment (start 151.5 70.75) (end 151.5 68) (width 0.25) (layer "B.Cu") (net 10))
   (segment (start 142.4 82.6) (end 140 82.6) (width 0.25) (layer "B.Cu") (net 10))
@@
   (segment (start 134.38 117.38) (end 151.87 117.38) (width 0.25) (layer "F.Cu") (net 18))
   (segment (start 119.54 99.3) (end 120.62 100.38) (width 1) (layer "F.Cu") (net 18))
-  (segment (start 120 99.76) (end 120.62 100.38) (width 0.25) (layer "F.Cu") (net 18))
   (segment (start 117 104) (end 117 105) (width 1) (layer "F.Cu") (net 18))
   (segment (start 99.38 101.38) (end 105 107) (width 0.25) (layer "F.Cu") (net 18))
@@
   (segment (start 148 105.62) (end 149.5 105.62) (width 0.25) (layer "F.Cu") (net 18))
   (segment (start 152.5 108.62) (end 149.5 105.62) (width 0.25) (layer "F.Cu") (net 18))
-  (segment (start 149.5 105.62) (end 149.62 105.62) (width 0.25) (layer "F.Cu") (net 18))
   (segment (start 129 112) (end 129 102) (width 1) (layer "F.Cu") (net 18))
   (segment (start 99.38 85) (end 99.38 101.38) (width 0.25) (layer "F.Cu") (net 18))
@@
   (segment (start 154 129) (end 170 129) (width 1) (layer "F.Cu") (net 48))
   (segment (start 174 123.46) (end 173.46 123.46) (width 1) (layer "F.Cu") (net 48))
-  (via (at 154 129) (size 0.8) (drill 0.4) (layers "F.Cu" "B.Cu") (net 48))
   (zone (net 7) (net_name "GND") (layer "B.Cu") (hatch edge 0.5)
     (connect_pads (clearance 0.5))
